File: design.kicad_pcb (KiCad board)
At the start: 4 copper layers, 43.2 x 50.8 mm, 75 parts, among them J1 STEREO, J2 USB_B_Micro, J3 2mm, P1 TSW-106-08-G-D-RA, P2 TSW-106-08-G-D-RA, U1 OPA354, U10 74LVC1G125, U11 74LVC1G125, U2 OPA354, U3 OPA354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

Commit message: Update
Parts:
- moved J3 5.46 mm to (138.3, 101.1)
- moved SP1 2.18 mm to (159.7, 110.4)
